Commit message: Modified sensor xacro files.

File: go_chase_it/catkin_ws/src/my_robot/urdf/diff_bot/accessories/depth_camera.urdf.xacro (robot description, xacro)
@@ -1,96 +1,95 @@
 <?xml version="1.0"?>
-<robot xmlns:xacro="http://ros.org/wiki/xacro">
-  <material name="Red_one">
-    <color rgba="0.8 0.0 0.0 1.0"/>
-  </material>
-  <xacro:macro name="depth_camera_mount" params="prefix topic parent_link">
-    <xacro:macro name="depth_camera" params=" frame:=camera topic:=camera h_fov:=1.5184351666666667 v_fov:=1.0122901111111111 min_range:=0.105 max_range:=8.0 width:=640 height:=480 update_rate:=30 robot_namespace:=/">
-      <!-- this link is the origin for the camera's data -->
-      <link name="${frame}" />
-      <!--
-        The gazebo plugin aligns the depth data with the Z axis, with X=left and Y=up
-        ROS expects the depth data along the X axis, with Y=left and Z=up
-        This link only exists to give the gazebo plugin the correctly-oriented frame
-      -->
-      <link name="${frame}_gazebo" />
-      <joint name="${frame}_gazebo_joint" type="fixed">
-        <parent link="${frame}"/>
-        <child link="${frame}_gazebo"/>
-        <origin xyz="0.0 0 0" rpy="-1.5707963267948966 0 -1.5707963267948966"/>
-      </joint>
-      <gazebo reference="${frame}">
-        <turnGravityOff>true</turnGravityOff>
-        <sensor type="depth" name="${prefix}_camera_depth">
-          <update_rate>${update_rate}</update_rate>
-          <camera>
-            <!-- 75x65 degree FOV for the depth sensor -->
-            <horizontal_fov>${h_fov}</horizontal_fov>
-            <vertical_fov>${v_fov}</vertical_fov>
-            <image>
-              <width>${width}</width>
-              <height>${height}</height>
-              <!-- TODO: check what format the camera hardware delivers and set this to match! -->
-              <format>R8G8B8</format>
-            </image>
-            <clip>
-              <!-- give the color sensor a maximum range of 50m so that the simulation renders nicely -->
-              <near>0.01</near>
-              <far>50.0</far>
-            </clip>
-          </camera>
-          <plugin name="kinect_controller" filename="libgazebo_ros_openni_kinect.so">
-            <baseline>0.2</baseline>
-            <alwaysOn>true</alwaysOn>
-            <updateRate>30.0</updateRate>
-            <cameraName>camera</cameraName>
-            <frameName>camera_rgb_optical_frame</frameName>
-            <imageTopicName>rgb/image_raw</imageTopicName>
-            <depthImageTopicName>depth/image_raw</depthImageTopicName>
-            <pointCloudTopicName>depth/points</pointCloudTopicName>
-            <cameraInfoTopicName>rgb/camera_info</cameraInfoTopicName>
-            <depthImageCameraInfoTopicName>depth/camera_info</depthImageCameraInfoTopicName>
-            <pointCloudCutoff>0.4</pointCloudCutoff>
-            <hackBaseline>0.07</hackBaseline>
-            <distortionK1>0.0</distortionK1>
-            <distortionK2>0.0</distortionK2>
-            <distortionK3>0.0</distortionK3>
-            <distortionT1>0.0</distortionT1>
-            <distortionT2>0.0</distortionT2>
-            <CxPrime>0.0</CxPrime>
-            <Cx>0.0</Cx>
-            <Cy>0.0</Cy>
-            <focalLength>0</focalLength>
-            <hackBaseline>0</hackBaseline>
-          </plugin>
-        </sensor>
-      </gazebo>
-    </xacro:macro>
-    <link name="${prefix}_camera_lens">
+<robot name="sensor_kinect" xmlns:xacro="http://ros.org/wiki/xacro">
+  <xacro:property name="kinect_cam_py" value="-0.0125"/>
+  <xacro:property name="M_PI" value="3.14159"/>
+  <xacro:macro name="sensor_kinect" params="parent">
+    <joint name="camera_rgb_joint" type="fixed">
+      <origin xyz="0.6 0 0.06" rpy="0 0 0"/>
+      <parent link="${parent}"/>
+      <child link="camera_rgb_frame" />
+    </joint>
+    <link name="camera_rgb_frame"/>
+    <joint name="camera_rgb_optical_joint" type="fixed">
+      <origin xyz="0 0 0" rpy="${-M_PI/2} 0 ${-M_PI/2}" />
+      <parent link="camera_rgb_frame" />
+      <child link="camera_rgb_optical_frame" />
+    </joint>
+    <link name="camera_rgb_optical_frame"/>
+    <joint name="camera_joint" type="fixed">
+      <origin xyz="-0.031 ${-kinect_cam_py} -0.016" rpy="0 0 0"/>
+      <parent link="camera_rgb_frame"/>
+      <child link="camera_link"/>
+    </joint>
+      <link name="camera_link">
       <visual>
-        <!--
-          the model's origin is in the middle & it's rotated to lie in
-          the optical standard with X left, Y up, and Z forward
-        -->
-        <origin xyz="0.0115 0 0.0100" rpy="0 0 0" />
+       <origin xyz="0 0 0" rpy="0 0 0"/>
         <geometry>
-          <!-- Origin of this mesh is the base of the bracket. -->
-          <!-- <mesh filename="package://my_robot/meshes/sick_lms-100.stl" /> -->
-          <!-- <box size=".4 .1 .1" /> -->
-          <mesh filename="package://my_robot/meshes/kinect.dae" />
+         <mesh filename="package://my_robot/meshes/kinect.dae"/>
         </geometry>
-        <material name="Red_one" />
+        <material name="Blue" />
       </visual>
+  	  <collision>
+        <origin xyz="0.0 0.0 0.0" rpy="0 0 0"/>
+  	    <geometry>
+  	      <box size="0.07271 0.27794 0.073"/>
+  	    </geometry>
+  	  </collision>
+      <inertial>
+        <mass value="0.564" />
+        <origin xyz="0 0 0" />
+        <inertia ixx="0.003881243" ixy="0.0" ixz="0.0"
+                 iyy="0.000498940" iyz="0.0"
+                 izz="0.003879257" />
+      </inertial>
     </link>
-    <joint type="fixed" name="${prefix}_camera_lens_joint">
-      <origin xyz="0 0 0" rpy="0 0 0" />
-      <parent link="${parent_link}" />
-      <child link="${prefix}_camera_lens" />
-    </joint>
-    <joint type="fixed" name="${prefix}_camera_joint">
-      <origin xyz="0.025 0 0" rpy="0 0 0" />
-      <parent link="${prefix}_camera_lens" />
-      <child link="${prefix}_camera" />
-    </joint>
-    <xacro:depth_camera frame="${prefix}_camera" topic="${topic}"/>
+	<joint name="camera_depth_joint" type="fixed">
+	  <origin xyz="0 ${2 * -kinect_cam_py} 0" rpy="0 0 0" />
+	  <parent link="camera_rgb_frame" />
+	  <child link="camera_depth_frame" />
+	</joint>
+	<link name="camera_depth_frame"/>
+	<joint name="camera_depth_optical_joint" type="fixed">
+	  <origin xyz="0 0 0" rpy="${-M_PI/2} 0 ${-M_PI/2}" />
+	  <parent link="camera_depth_frame" />
+	  <child link="camera_depth_optical_frame" />
+	</joint>
+	<link name="camera_depth_optical_frame"/>
+	<!-- Kinect sensor for simulation -->
+    <gazebo reference="camera_link">
+      <sensor type="depth" name="camera">
+        <always_on>true</always_on>
+        <update_rate>20.0</update_rate>
+        <camera>
+          <horizontal_fov>${60.0*M_PI/180.0}</horizontal_fov>
+          <image>
+            <format>B8G8R8</format>
+            <width>640</width>
+            <height>480</height>
+          </image>
+          <clip>
+            <near>0.05</near>
+            <far>20.0</far>
+          </clip>
+        </camera>
+        <plugin name="kinect_camera_controller" filename="libgazebo_ros_openni_kinect.so">
+          <cameraName>camera</cameraName>
+          <alwaysOn>true</alwaysOn>
+          <updateRate>10</updateRate>
+          <imageTopicName>rgb/image_raw</imageTopicName>
+          <depthImageTopicName>depth/image_raw</depthImageTopicName>
+          <pointCloudTopicName>depth/points</pointCloudTopicName>
+          <cameraInfoTopicName>rgb/camera_info</cameraInfoTopicName>
+          <depthImageCameraInfoTopicName>depth/camera_info</depthImageCameraInfoTopicName>
+          <frameName>camera_depth_optical_frame</frameName>
+          <baseline>0.1</baseline>
+          <distortion_k1>0.0</distortion_k1>
+          <distortion_k2>0.0</distortion_k2>
+          <distortion_k3>0.0</distortion_k3>
+          <distortion_t1>0.0</distortion_t1>
+          <distortion_t2>0.0</distortion_t2>
+          <pointCloudCutoff>0.4</pointCloudCutoff>
+        </plugin>
+      </sensor>
+    </gazebo>
   </xacro:macro>
 </robot>

File: go_chase_it/catkin_ws/src/my_robot/urdf/diff_bot/skid_steer_diff_bot_base_laser.urdf.xacro (robot description, xacro)
@@ -83,10 +83,4 @@
     <xacro:plate parent="${plate1_parent}" suffix="plate1" parent_size_z="${plate1_parent_size_z}" plate_x="${plate1_x}" plate_y="${plate1_y}"
     plate_z="${plate1_z}" color_rviz="OffWhite" color_gazebo="WoodFloor" />
-    <link name="camera_mountpoint"/>
-    <joint name="camera_mountpoint_joint" type="fixed">
-      <origin xyz="${base_size_x/2} 0 .05" rpy="0 0 0" />
-      <parent link="${plate1_parent}_plate1_plate_link"/>
-      <child link="camera_mountpoint" />
-    </joint>
-    <xacro:depth_camera_mount prefix="custom" topic="image" parent_link="camera_mountpoint"/>
+    <xacro:sensor_kinect parent="${plate1_parent}_plate1_plate_link"/>
 </robot>
